File: kurage.kicad_pcb (KiCad board)
At the start: 2 copper layers, 346.5 x 118.1 mm, 106 parts, among them SW1 ESC, SW10 R, SW11 Y, SW12 I, SW13 P, SW14 ], SW15 UNDEFINED2, SW16 CTRL, SW17 A, SW18 D, SW19 G, SW2 Q, SW20 J, SW21 L, SW22 ', SW23 S, SW24 F, SW25 H, SW26 K, SW27 ;, SW28 ENTER, SW29 UNDEFINED3, SW3 E, SW30 LSHIFT, SW31 Z, SW32 C, SW33 B, SW34 M, SW35 ., SW36 RSHIFT, SW37 X, SW38 V, SW39 N, SW4 T, SW40 ,, SW41 /, SW42 UP, SW43 LOWER, SW44 UNDEFINED1, SW45 WIN, SW46 RAISE, SW47 LEFT, SW48 RIGHT, SW49 LSPACE, SW5 U, SW50 RSPACE, SW51 ALT, SW52 DOWN, SW6 O, SW7 [, SW8 BACKSPACE, SW9 W, U1 ProMicro

Commit message: progress
Parts:
- added G***: LOGO, rin:kurage_wob_test, F.Cu at (28.8, 59.1)
- added Ref**: Val**, kbd:M2_HOLE, F.Cu at (264.7, 92.2)
- added Ref**: Val**, kbd:M2_HOLE, F.Cu at (324.4, 97.5)
- added Ref**: Val**, kbd:M2_HOLE, F.Cu at (192.0, 133.1)
- added Ref**: Val**, kbd:M2_HOLE, F.Cu at (124.9, 65.5)
- added Ref**: Val**, kbd:M2_HOLE, F.Cu at (78.7, 133.2)
- added Ref**: Val**, kbd:M2_HOLE, F.Cu at (-6.10, 90.7)
- added Ref**: Val**, kbd:M2_HOLE_v2, F.Cu at (271.5, 66.1)
- added Ref**: Val**, kbd:M2_HOLE_v2, F.Cu at (201.5, 133.2)
Connections:
- U1 pad 1: ROW6 -> ROW7
- U1 pad 2: ROW7 -> ROW6
Routing:
- net ROW7: track 438.6 -> 449.2 mm, vias 2 -> 0
- net ROW6: track 451.5 -> 453.7 mm
- net ROW3: track 393.8 -> 394.8 mm
- added copper zone on F.Cu, net (none)

Commit message: update
Parts:
- G***: footprint rin:kurage_wob_test -> rin:kurage_wob
Changed lines of the file:
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@@
     (add_net GND)
   )
-  (module kbd:M2_HOLE (layer F.Cu)
-    (at 264.668 92.202)
-    (descr "Mounting Hole 2.2mm, no annular, M2")
-    (tags "mounting hole 2.2mm no annular m2")
-    (attr virtual)
-    (fp_text reference Ref** (at -0.95 -0.55) (layer F.Fab) hide
-      (effects (font (size 1 1) (thickness 0.15)))
-    )
-    (fp_text value Val** (at 0 0.55) (layer F.Fab) hide
-      (effects (font (size 1 1) (thickness 0.15)))
-    )
-    (pad "" thru_hole circle (at 0 0) (size 6.5 6.5) (drill 4.2) (layers *.Cu *.Mask))
-  )
-  (module kbd:M2_HOLE (layer F.Cu)
-    (at 324.438515 97.536 8)
-    (descr "Mounting Hole 2.2mm, no annular, M2")
-    (tags "mounting hole 2.2mm no annular m2")
-    (attr virtual)
-    (fp_text reference Ref** (at -0.95 -0.55 8) (layer F.Fab) hide
-      (effects (font (size 1 1) (thickness 0.15)))
-    )
-    (fp_text value Val** (at 0 0.55 8) (layer F.Fab) hide
-      (effects (font (size 1 1) (thickness 0.15)))
-    )
-    (pad "" thru_hole circle (at 0 0 8) (size 6.5 6.5) (drill 4.2) (layers *.Cu *.Mask))
-  )
-  (module kbd:M2_HOLE (layer F.Cu)
-    (at 191.997648 133.089334)
-    (descr "Mounting Hole 2.2mm, no annular, M2")
-    (tags "mounting hole 2.2mm no annular m2")
-    (attr virtual)
-    (fp_text reference Ref** (at -0.95 -0.55) (layer F.Fab) hide
-      (effects (font (size 1 1) (thickness 0.15)))
-    )
-    (fp_text value Val** (at 0 0.55) (layer F.Fab) hide
-      (effects (font (size 1 1) (thickness 0.15)))
-    )
-    (pad "" thru_hole circle (at 0 0) (size 6.5 6.5) (drill 4.2) (layers *.Cu *.Mask))
-  )
-  (module kbd:M2_HOLE (layer F.Cu)
-    (at 124.907871 65.532)
-    (descr "Mounting Hole 2.2mm, no annular, M2")
-    (tags "mounting hole 2.2mm no annular m2")
-    (attr virtual)
-    (fp_text reference Ref** (at -0.95 -0.55) (layer F.Fab) hide
-      (effects (font (size 1 1) (thickness 0.15)))
-    )
-    (fp_text value Val** (at 0 0.55) (layer F.Fab) hide
-      (effects (font (size 1 1) (thickness 0.15)))
-    )
-    (pad "" thru_hole circle (at 0 0) (size 6.5 6.5) (drill 4.2) (layers *.Cu *.Mask))
-  )
-  (module kbd:M2_HOLE (layer F.Cu)
-    (at 78.68158 133.23062)
-    (descr "Mounting Hole 2.2mm, no annular, M2")
-    (tags "mounting hole 2.2mm no annular m2")
-    (attr virtual)
-    (fp_text reference Ref** (at -0.95 -0.55) (layer F.Fab) hide
-      (effects (font (size 1 1) (thickness 0.15)))
-    )
-    (fp_text value Val** (at 0 0.55) (layer F.Fab) hide
-      (effects (font (size 1 1) (thickness 0.15)))
-    )
-    (pad "" thru_hole circle (at 0 0) (size 6.5 6.5) (drill 4.2) (layers *.Cu *.Mask))
-  )
-  (module kbd:M2_HOLE (layer F.Cu)
-    (at -6.096 90.678)
-    (descr "Mounting Hole 2.2mm, no annular, M2")
-    (tags "mounting hole 2.2mm no annular m2")
-    (attr virtual)
-    (fp_text reference Ref** (at -0.95 -0.55) (layer F.Fab) hide
-      (effects (font (size 1 1) (thickness 0.15)))
-    )
-    (fp_text value Val** (at 0 0.55) (layer F.Fab) hide
-      (effects (font (size 1 1) (thickness 0.15)))
-    )
-    (pad "" thru_hole circle (at 0 0) (size 6.5 6.5) (drill 4.2) (layers *.Cu *.Mask))
-  )
-  (module kbd:M2_HOLE_v2 (layer F.Cu)
-    (at 271.47774 66.09588)
-    (descr "Mounting Hole 2.2mm, no annular, M2")
-    (tags "mounting hole 2.2mm no annular m2")
-    (attr virtual)
-    (fp_text reference Ref** (at -0.95 -0.55) (layer F.Fab) hide
-      (effects (font (size 1 1) (thickness 0.15)))
-    )
-    (fp_text value Val** (at 0 0.55) (layer F.Fab) hide
-      (effects (font (size 1 1) (thickness 0.15)))
-    )
-    (pad "" np_thru_hole circle (at 0 0) (size 4.2 4.2) (drill 4.2) (layers *.Cu *.Mask))
-  )
-  (module rin:kurage_wob_test (layer F.Cu)
+  (module rin:kurage_wob (layer F.Cu)
     (at 28.83154 59.11596)
     (fp_text reference G*** (at 0 0) (layer F.SilkS) hide
@@
       (xy 2.511465 -91.480531)) (layer F.Mask) (width 0.01))
   )
+  (module kbd:M2_HOLE (layer F.Cu)
+    (at 264.668 92.202)
+    (descr "Mounting Hole 2.2mm, no annular, M2")
+    (tags "mounting hole 2.2mm no annular m2")
+    (attr virtual)
+    (fp_text reference Ref** (at -0.95 -0.55) (layer F.Fab) hide
+      (effects (font (size 1 1) (thickness 0.15)))
+    )
+    (fp_text value Val** (at 0 0.55) (layer F.Fab) hide
+      (effects (font (size 1 1) (thickness 0.15)))
+    )
+    (pad "" thru_hole circle (at 0 0) (size 6.5 6.5) (drill 4.2) (layers *.Cu *.Mask))
+  )
+  (module kbd:M2_HOLE (layer F.Cu)
+    (at 324.438515 97.536 8)
+    (descr "Mounting Hole 2.2mm, no annular, M2")
+    (tags "mounting hole 2.2mm no annular m2")
+    (attr virtual)
+    (fp_text reference Ref** (at -0.95 -0.55 8) (layer F.Fab) hide
+      (effects (font (size 1 1) (thickness 0.15)))
+    )
+    (fp_text value Val** (at 0 0.55 8) (layer F.Fab) hide
+      (effects (font (size 1 1) (thickness 0.15)))
+    )
+    (pad "" thru_hole circle (at 0 0 8) (size 6.5 6.5) (drill 4.2) (layers *.Cu *.Mask))
+  )
+  (module kbd:M2_HOLE (layer F.Cu)
+    (at 191.997648 133.089334)
+    (descr "Mounting Hole 2.2mm, no annular, M2")
+    (tags "mounting hole 2.2mm no annular m2")
+    (attr virtual)
+    (fp_text reference Ref** (at -0.95 -0.55) (layer F.Fab) hide
+      (effects (font (size 1 1) (thickness 0.15)))
+    )
+    (fp_text value Val** (at 0 0.55) (layer F.Fab) hide
+      (effects (font (size 1 1) (thickness 0.15)))
+    )
+    (pad "" thru_hole circle (at 0 0) (size 6.5 6.5) (drill 4.2) (layers *.Cu *.Mask))
+  )
+  (module kbd:M2_HOLE (layer F.Cu)
+    (at 124.907871 65.532)
+    (descr "Mounting Hole 2.2mm, no annular, M2")
+    (tags "mounting hole 2.2mm no annular m2")
+    (attr virtual)
+    (fp_text reference Ref** (at -0.95 -0.55) (layer F.Fab) hide
+      (effects (font (size 1 1) (thickness 0.15)))
+    )
+    (fp_text value Val** (at 0 0.55) (layer F.Fab) hide
+      (effects (font (size 1 1) (thickness 0.15)))
+    )
+    (pad "" thru_hole circle (at 0 0) (size 6.5 6.5) (drill 4.2) (layers *.Cu *.Mask))
+  )
+  (module kbd:M2_HOLE (layer F.Cu)
+    (at 78.68158 133.23062)
+    (descr "Mounting Hole 2.2mm, no annular, M2")
+    (tags "mounting hole 2.2mm no annular m2")
+    (attr virtual)
+    (fp_text reference Ref** (at -0.95 -0.55) (layer F.Fab) hide
+      (effects (font (size 1 1) (thickness 0.15)))
+    )
+    (fp_text value Val** (at 0 0.55) (layer F.Fab) hide
+      (effects (font (size 1 1) (thickness 0.15)))
+    )
+    (pad "" thru_hole circle (at 0 0) (size 6.5 6.5) (drill 4.2) (layers *.Cu *.Mask))
+  )
+  (module kbd:M2_HOLE (layer F.Cu)
+    (at -6.096 90.678)
+    (descr "Mounting Hole 2.2mm, no annular, M2")
+    (tags "mounting hole 2.2mm no annular m2")
+    (attr virtual)
+    (fp_text reference Ref** (at -0.95 -0.55) (layer F.Fab) hide
+      (effects (font (size 1 1) (thickness 0.15)))
+    )
+    (fp_text value Val** (at 0 0.55) (layer F.Fab) hide
+      (effects (font (size 1 1) (thickness 0.15)))
+    )
+    (pad "" thru_hole circle (at 0 0) (size 6.5 6.5) (drill 4.2) (layers *.Cu *.Mask))
+  )
   (module kbd:M2_HOLE_v2 (layer F.Cu)
+    (at 271.47774 66.09588)
+    (descr "Mounting Hole 2.2mm, no annular, M2")
+    (tags "mounting hole 2.2mm no annular m2")
+    (attr virtual)
+    (fp_text reference Ref** (at -0.95 -0.55) (layer F.Fab) hide
+      (effects (font (size 1 1) (thickness 0.15)))
+    )
+    (fp_text value Val** (at 0 0.55) (layer F.Fab) hide
+      (effects (font (size 1 1) (thickness 0.15)))
+    )
+    (pad "" np_thru_hole circle (at 0 0) (size 4.2 4.2) (drill 4.2) (layers *.Cu *.Mask))
+  )
+  (module kbd:M2_HOLE_v2 (layer F.Cu)

Commit message: backup
Parts:
- removed the Ref** at (271.5, 66.1)
- added Ref**: Val**, kbd:M2_HOLE, F.Cu at (270.6, 66.9)
- added Ref**: Val**, kbd:M2_HOLE, F.Cu at (17.0, 65.0)
- moved Ref** 38.1 mm to (27.2, 109.2)
- moved Ref** 36.7 mm to (230.9, 106.4)
- moved Ref** 0.31 mm to (324.4, 97.8)
Routing:
- net COL1: track 187.8 -> 189.3 mm
- net Net-(D9-Pad2): track 7.00 -> 5.71 mm
- net COL2: track 361.0 -> 362.2 mm
- net COL3: track 641.1 -> 642.1 mm

Commit message: curved traces
Parts:
- G***: footprint rin:kurage_wob -> rin:kurage_bow
Routing:
- net COL7: track 414.0 -> 392.3 mm
- net COL4: track 441.9 -> 449.7 mm
- net COL2: track 362.2 -> 369.9 mm
- net COL6: track 450.1 -> 456.2 mm
- net ROW3: track 394.8 -> 400.5 mm
- net ROW7: track 449.2 -> 454.0 mm
- net COL1: track 189.3 -> 193.9 mm
- net COL5: track 365.0 -> 361.0 mm
- net ROW5: track 390.1 -> 392.9 mm
- net COL0: track 81.6 -> 83.8 mm
- net ROW0: track 357.7 -> 356.0 mm
- net ROW1: track 328.5 -> 327.0 mm
- net ROW2: track 329.0 -> 330.0 mm
- net ROW4: track 358.7 -> 357.9 mm
- net Net-(D48-Pad2): track 17.1 -> 16.4 mm
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Other:
- board text added: "rev0"
